File: Schematic1.sch (EAGLE design)
At the start: 58 parts, among them Q1 500mA, Q2 500mA, Q3 500mA, U1 HX711, U2 HX711, U3 5V, U4 STM32F0XXC1T, U5 PCF8574T/3,512SOT162-1-M, U6 HX711, U7 3.3V/150mA

Commit message: Add files via upload
Final Main Hub PCB schematic and layout to be checked
Parts:
- removed C13, C15, C16: 2.2uF, SparkFun-Capacitors:2.2UF-0603-10V-20%
- removed C14, C17: 470pF, SparkFun-Capacitors:470PF-0603-50V-5%
- removed D1, D2, D3: (no value), SparkFun-LED:LED5MM
- removed JP1, JP2, JP3, JP6, JP8: (no value), pinhead:PINHD-1X6
- removed JP7: (no value), pinhead:PINHD-1X9
- removed R13, R14, R15: (no value), SparkFun-Resistors:RESISTOR0603
- added BPV3, BPV5: 470pF, SparkFun-Capacitors:0.33UF/330NF-0805-50V-10%
- added BUTTPINS, LEDS, PRGPIN: (no value), pinhead:PINHD-1X6
- added DCB1, DCB2, DCB3, DCLCD, DCLD1, DCLD2, DCLD3, DCM1, DCM24, DCM36, DCM48, DCM9, DCO1, DCO2, DCSW: 0.33µF, SparkFun-Capacitors:0.33UF/330NF-0805-50V-10%
- added DCV3, DCV5, DCXB: 2.2µF, SparkFun-Capacitors:0.33UF/330NF-0805-50V-10%
- added J2: (no value), SparkFun-Connectors:JST_2MM_MALE
- added LCD: (no value), pinhead:PINHD-1X10
- added LOAD1, LOAD2, LOAD3: (no value), pinhead:PINHD-1X4
- added RB1, RB2, RB3, RLD1, RLD2, RLD3: 1k, SparkFun-Resistors:RESISTOR0805
- added RSW: 10k, SparkFun-Resistors:RESISTOR0805
- added VR1: 10k, SparkFun-Resistors:TRIMPOT-PTH-10MM-KNOB-1/2W-10%
- C1, C10, C2, C5, C6, C9: value 10uF -> 10µF; device SparkFun-Capacitors:10UF-0603-6.3V-20% -> SparkFun-Capacitors:0.33UF/330NF-0805-50V-10%
- C11, C12, C3, C4, C7, C8: value 0.1uF -> 0.1µF; device SparkFun-Capacitors:0.1UF-0603-25V-(+80/-20%) -> SparkFun-Capacitors:0.33UF/330NF-0805-50V-10%
- Q1, Q2, Q3: value 500mA -> 600mA/40V; device SparkFun-DiscreteSemi:TRANS_PNP_RES-DDTB142TC -> SparkFun-DiscreteSemi:TRANS_PNP-MMBT4403
- R1, R10, R11, R12, R2, R3, R4, R5, R6, R7, R8, R9: device SparkFun-Resistors:RESISTOR0603 -> SparkFun-Resistors:RESISTOR0805
- R16, R17: value (none) -> 4.7k; device SparkFun-Resistors:RESISTOR0603 -> SparkFun-Resistors:RESISTOR0805
- renumbered JP4 to RFID, JP5 to XBEE, U3 to VR5, U7 to VR3
Connections:
- net N$38 renamed PWR_IN
- removed net A13: JP8.2, U4A.PA13
- removed net A14: JP8.3, U4A.PA14
- removed net N$39: D1.C, R13.1
- removed net N$41: D2.C, R14.1
- removed net N$42: D3.C, R15.1
- removed net VCC: C1.1, C15.1, C5.1, C9.1, JP7.1, JP8.1, Q1.E, Q2.E, Q3.E, R16.2, R17.2, RFID.1, U1.DVDD, U1.VSUP, U2.DVDD, U2.VSUP, U5.VDD, U6.DVDD, U6.VSUP, XBEE.1
- new net A: U5.P3, VR1.CCW
- new net B: LCD.9, VR1.WIPER
- new net GND_IN: J2.-, VR3.GND, VR5.GND
- new net N$1: J1.-, J2.+
- new net N$35: BUTTPINS.1, DCB1.1, RB1.2
- new net N$38: BUTTPINS.5, DCB3.1, RB3.2
- new net P3V: C1.1, C5.1, C9.1, DCM1.2, DCM24.2, DCM36.2, DCM48.2, DCM9.2, DCV3.1, DCXB.1, PRGPIN.1, Q1.E, Q2.E, Q3.E, R16.2, R17.2, RFID.1, RSW.1, U1.DVDD, U1.VSUP, U2.DVDD, U2.VSUP, U4B.VDD, U4B.VDDA, U4B.VDD_2, U4B.VDD_3, U4B.VDD_4, U6.DVDD, U6.VSUP, VR3.OUT, XBEE.1
- new net P5V: DCLCD.2, DCV5.1, LCD.1, U5.VDD, VR5.OUT
- new net RST: DCSW.2, PRGPIN.5, RSW.2, S1.1, U4A.NRST
- new net SWCLK: PRGPIN.2, U4A.PA14
- new net SWDIO: PRGPIN.4, U4A.PA13
- net A0: now also RB1.1; no longer JP3.1
- net A1: now also RB2.1; no longer JP3.3
- net A10: now also RLD3.1; no longer D3.A
- net A11: now also RB3.1; no longer JP3.5
- net A8: now also RLD1.1; no longer D1.A
- net A9: now also RLD2.1; no longer D2.A
- net D0: now also LCD.8; no longer JP7.8
- net D1: now also LCD.7; no longer JP7.7
- net D2: now also LCD.6; no longer JP7.6
- net D4: now also LCD.5; no longer JP7.5
- net D5: now also LCD.4; no longer JP7.4
- net D6: now also LCD.3; no longer JP7.3
- net D7: now also LCD.2; no longer JP7.2
- net GND: now also BPV3.2, BPV5.2, BUTTPINS.2, BUTTPINS.4, BUTTPINS.6, DCB1.2, DCB2.2, DCB3.2, DCLCD.1, DCLD1.2, DCLD2.2, DCLD3.2, DCM1.1, DCM24.1, DCM36.1, DCM48.1, DCM9.1, DCO1.2, DCO2.2, DCSW.1, DCV3.2, DCV5.2, DCXB.2, LCD.10, LEDS.2, LEDS.4, LEDS.6, LOAD1.2, LOAD2.2, LOAD3.2, PRGPIN.3, VR1.CW; no longer C13.2, C14.2, C15.2, C16.2, C17.2, JP1.2, JP2.2, JP3.2, JP3.4, JP3.6, JP6.2, JP7.9, JP8.6, R13.2, R14.2, R15.2
- net N$10: now also DCLD1.1, LEDS.1, RLD1.2; no longer S1.1, U4A.NRST
- net N$12: now also LOAD3.3; no longer JP6.3
- net N$13: now also LOAD3.4; no longer JP6.4
- net N$17: now also LOAD3.1; no longer JP6.1
- net N$2: now also LOAD2.3; no longer JP1.3
- net N$21: now also DCO1.1
- net N$22: now also DCO2.1
- net N$23: now also LOAD1.3; no longer JP2.3
- net N$24: now also LOAD1.4; no longer JP2.4
- net N$28: now also LOAD1.1; no longer JP2.1
- net N$3: now also LOAD2.4; no longer JP1.4
- net N$32: now also DCLD2.1, LEDS.3, RLD2.2; no longer J1.-, VR3.GND, VR5.GND
- net N$33: now also DCLD3.1, LEDS.5, RLD3.2; no longer C16.1, VR3.OUT
- net N$34: now also BPV3.1; no longer C17.1
- net N$36: now also BUTTPINS.3, DCB2.1, RB2.2; no longer C13.1, U4B.VDD, U4B.VDDA, U4B.VDD_2, U4B.VDD_3, U4B.VDD_4, VR5.OUT
- net N$37: now also BPV5.1; no longer C14.1
- net N$7: now also LOAD2.1; no longer JP1.1
Other:
- note added: "LCD Out Pins"
- note added: "Load Cell 1 in"
- note added: "Load Cell 2 in"
- note added: "Load Cell 3 in"
- note added: "Programming Pins"
