File: Central Hub.brd (EAGLE design)
At the start: 70 x 80.3 mm, 59 parts, among them Q1 500mA, Q2 500mA, Q3 500mA, U1 HX711, U2 HX711, U3 5V, U4 STM32F0XXC1T, U5 PCF8574T/3,512SOT162-1-M, U6 HX711, U7 3.3V/150mA

Commit message: final stuff
Parts:
- added C18, C19, C20: 0.33µF, SparkFun-Capacitors:0805
- C13, C15, C16: value 2.2uF -> 0.33µF; device SparkFun-Capacitors:0603 -> SparkFun-Capacitors:0805
- C9: value 10uF -> 0.33µF; device SparkFun-Capacitors:0603 -> SparkFun-Capacitors:0805
Connections:
- removed net N$10: S1.1, U4.7
- new net N$1: C20.1, S1.1, U4.7
- net GND: now also C18.2, C19.2, C20.2; no longer U4.44
- net N$21: now also C19.1
- net N$22: now also C18.1
Routing:
- net N$10: track 27.5 -> 0.00 mm
- net P3V: track 219.8 -> 217.9 mm
