File: MainHubPCB.sch (EAGLE design)
At the start: 77 parts, among them Q1 600mA/40V, Q2 600mA/40V, Q3 600mA/40V, U1 HX711, U2 HX711, U4 STM32F0XXC1T, U5 PCF8574T/3,512SOT162-1-M, U6 HX711

Commit message: final stuff
Parts:
- removed LCD: (no value), pinhead:PINHD-1X10
- added LCDJMP: (no value), jumper:JP2E
- added LCDPINS: (no value), pinhead:PINHD-1X12
- renumbered Y1 to OSC
Connections:
- net A2 renamed TX
- net A3 renamed RX
- net B6 renamed SCL
- net B7 renamed SDA
- net N$12 renamed 3_A-
- net N$13 renamed 3_A+
- net N$17 renamed 3_VDD
- net N$2 renamed 2_A-
- net N$23 renamed 1_A-
- net N$24 renamed 1_A+
- net N$28 renamed 1_VDD
- net N$3 renamed 2_A+
- net N$7 renamed 2_VDD
- removed net B: LCD.9, VR1.WIPER
- removed net D0: LCD.8, U5.P0
- removed net D1: LCD.7, U5.P1
- removed net D2: LCD.6, U5.P2
- new net E: LCDPINS.7, U5.P2
- new net POT_A: U5.P3, VR1.CCW
- new net POT_B: LCDPINS.10, VR1.WIPER
- new net RS: LCDPINS.9, U5.P0
- new net RW: LCDPINS.8, U5.P1
- net A: now also LCDJMP.2, LCDPINS.2; no longer U5.P3, VR1.CCW
- net D4: now also LCDPINS.6; no longer LCD.5
- net D5: now also LCDPINS.5; no longer LCD.4
- net D6: now also LCDPINS.4; no longer LCD.3
- net D7: now also LCDPINS.3; no longer LCD.2
- net GND: now also LCDPINS.1, LCDPINS.12; no longer LCD.10
- net P3V: now also LCDJMP.1
- net P5V: now also LCDJMP.3, LCDPINS.11; no longer LCD.1
Other:
- moved on the sheet: VR1
