File: Player Module.sch (EAGLE design)
At the start: 25 parts, among them U3 5V, U4 STM32F0XXC1T, U5 PCF8574T/3,512SOT162-1-M, U7 3.3V/150mA

Commit message: updates as of wednesday night
Parts:
- removed C13, C15, C16: 2.2uF, SparkFun-Capacitors:2.2UF-0603-10V-20%
- removed C14, C17: 470pF, SparkFun-Capacitors:470PF-0603-50V-5%
- removed C9: 10uF, SparkFun-Capacitors:10UF-0603-6.3V-20%
- removed D1, D2, D3: (no value), SparkFun-LED:LED5MM
- removed J1: (no value), SparkFun-Connectors:JST_2MM_MALE
- removed JP5: (no value), pinhead:PINHD-1X4
- removed JP7: (no value), pinhead:PINHD-1X9
- removed R13, R14, R15, R16, R17: (no value), SparkFun-Resistors:RESISTOR0603
- removed U3: 5V, SparkFun-IC-Power:V_REG_MIC52055V
- removed U7: 3.3V/150mA, SparkFun-IC-Power:V_REG_MIC52053.3V
- added BPV3, BPV5: 470pF, SparkFun-Capacitors:0.33UF/330NF-0805-50V-10%
- added DCB1, DCB2, DCB3, DCD, DCL1, DCL2, DCL3, DCM1, DCM24, DCM36, DCM48, DCM9, DCO1, DCO2, DCSW, DCZ: 0.33µF, SparkFun-Capacitors:0.33UF/330NF-0805-50V-10%
- added DCV3, DCV5: 2.2µF, SparkFun-Capacitors:0.33UF/330NF-0805-50V-10%
- added JST1, JST2: (no value), SparkFun-Connectors:JST_2MM_MALE
- added LCD: (no value), pinhead:PINHD-1X10
- added LEDS: (no value), pinhead:PINHD-1X6
- added POT: 10k, SparkFun-Resistors:TRIMPOT-PTH-10MM-KNOB-1/2W-10%
- added RB4, RB5, RB6, RLD1, RLD2, RLD3: 1k, SparkFun-Resistors:RESISTOR0805
- added RD1, RD2: 4.7k, SparkFun-Resistors:RESISTOR0805
- added RSW: 10k, SparkFun-Resistors:RESISTOR0805
- added U$1: XB24-BPIT-004, XB24-BPIT-004:XB24-BPIT-004
- added VR3: 3.3V/150mA, SparkFun-IC-Power:V_REG_MIC52053.3V
- added VR5: 5V, SparkFun-IC-Power:V_REG_MIC52055V
- renumbered JP3 to BUTTPINS, JP8 to PRG, Y1 to OSC
Connections:
- removed net A13: PRG.2, U4A.PA13
- removed net A14: PRG.3, U4A.PA14
- removed net D0: JP7.8, U5.P0
- removed net D1: JP7.7, U5.P1
- removed net D2: JP7.6, U5.P2
- removed net D4: JP7.5, U5.P4
- removed net D5: JP7.4, U5.P5
- removed net D6: JP7.3, U5.P6
- removed net D7: JP7.2, U5.P7
- removed net N$32: J1.-, U3.GND, U7.GND
- removed net N$38: J1.+, U3.IN, U7.IN
- removed net N$39: D1.C, R13.1
- removed net N$41: D2.C, R14.1
- removed net N$42: D3.C, R15.1
- new net GND_IN: JST2.-, VR3.GND, VR5.GND
- new net N$1: JST1.-, JST2.+
- new net N$11: LCD.4, U5.P5
- new net N$12: LCD.5, U5.P4
- new net N$13: BUTTPINS.3, DCB2.1, RB5.2
- new net N$14: LCD.6, U5.P2
- new net N$15: LCD.7, U5.P1
- new net N$16: LCD.8, U5.P0
- new net N$17: BUTTPINS.5, DCB3.1, RB6.2
- new net N$3: DCL3.1, LEDS.1, RLD1.2
- new net N$4: DCL2.1, LEDS.3, RLD2.2
- new net N$5: DCL1.1, LEDS.5, RLD3.2
- new net N$8: BUTTPINS.1, DCB1.1, RB4.2
- new net N$9: LCD.2, U5.P7
- new net POT_A: POT.CCW, U5.P3
- new net POT_B: LCD.9, POT.WIPER
- new net PWR_IN: JST1.+, VR3.IN, VR5.IN
- new net RST: DCSW.1, PRG.5, RSW.2, S1.1, U4A.NRST
- new net SWCLK: PRG.2, U4A.PA14
- new net SWDIO: PRG.4, U4A.PA13
- net A0: now also RB4.1; no longer BUTTPINS.1
- net A1: now also RB5.1; no longer BUTTPINS.3
- net A10: now also RLD3.1; no longer D3.A
- net A11: now also RB6.1; no longer BUTTPINS.5
- net A2: now also U$1.2; no longer JP5.2
- net A3: now also U$1.3; no longer JP5.3
- net A8: now also RLD1.1; no longer D1.A
- net A9: now also RLD2.1; no longer D2.A
- net B6: now also RD1.1; no longer R16.1
- net B7: now also RD2.1; no longer R17.1
- net GND: now also BPV3.2, BPV5.2, DCB1.2, DCB2.2, DCB3.2, DCD.2, DCL1.2, DCL2.2, DCL3.2, DCM1.1, DCM24.1, DCM36.1, DCM48.1, DCM9.1, DCO1.2, DCO2.2, DCSW.2, DCV3.2, DCV5.2, DCZ.2, LCD.10, LEDS.2, LEDS.4, LEDS.6, POT.CW, PRG.3, U$1.10; no longer C13.2, C14.2, C15.2, C16.2, C17.2, C9.2, JP5.4, JP7.9, PRG.6, R13.2, R14.2, R15.2
- net N$10: now also LCD.3, U5.P6; no longer S1.1, U4A.NRST
- net N$21: now also DCO2.1
- net N$22: now also DCO1.1
- net N$34: now also BPV3.1, VR3.BP; no longer C17.1, U7.BP
- net N$37: now also BPV5.1, VR5.BP; no longer C14.1, U3.BP
- net P3.3V: now also DCM1.2, DCM24.2, DCM36.2, DCM48.2, DCM9.2, DCV3.1, DCZ.1, RD1.2, RD2.2, RSW.1, U$1.1, VR3.OUT; no longer C15.1, C16.1, C9.1, JP5.1, U7.OUT
- net P5V: now also DCD.1, DCV5.1, LCD.1, VR5.OUT; no longer C13.1, JP7.1, R16.2, R17.2, U3.OUT
Other:
- moved on the sheet: S1, U4B

Commit message: final stuff
Parts:
- removed LCD: (no value), pinhead:PINHD-1X10
- added LCDJMP: (no value), jumper:JP2E
- added LCDPINS: (no value), pinhead:PINHD-1X12
- renumbered U$1 to XBEE, U4 to STM32, U5 to PCFI2C
Connections:
- net A0 renamed PA0
- net A1 renamed PA1
- net A10 renamed PA10
- net A11 renamed PA11
- net A8 renamed PA8
- net A9 renamed PA9
- net B6 renamed SCL
- net B7 renamed SDA
- removed net A2: STM32A.PA2, XBEE.2
- removed net A3: STM32A.PA3, XBEE.3
- removed net A4: STM32A.PA4
- removed net A5: STM32A.PA5
- removed net A6: STM32A.PA6
- removed net A7: STM32A.PA7
- removed net N$10: LCD.3, PCFI2C.P6
- removed net N$11: LCD.4, PCFI2C.P5
- removed net N$12: LCD.5, PCFI2C.P4
- removed net N$14: LCD.6, PCFI2C.P2
- removed net N$15: LCD.7, PCFI2C.P1
- removed net N$16: LCD.8, PCFI2C.P0
- removed net N$9: LCD.2, PCFI2C.P7
- new net A: LCDJMP.2, LCDPINS.2
- new net D4: LCDPINS.6, PCFI2C.P4
- new net D5: LCDPINS.5, PCFI2C.P5
- new net D6: LCDPINS.4, PCFI2C.P6
- new net D7: LCDPINS.3, PCFI2C.P7
- new net E: LCDPINS.7, PCFI2C.P2
- new net RS: LCDPINS.9, PCFI2C.P0
- new net RW: LCDPINS.8, PCFI2C.P1
- new net RX: STM32A.PA2, XBEE.3
- new net TX: STM32A.PA3, XBEE.2
- net GND: now also LCDPINS.1, LCDPINS.12; no longer LCD.10
- net P3.3V: now also LCDJMP.1
- net P5V: now also LCDJMP.3, LCDPINS.11; no longer LCD.1
- net POT_B: now also LCDPINS.10; no longer LCD.9
Other:
- moved on the sheet: DCD
